File: plate/discipline-pcb.kicad_pcb (KiCad board)
At the start: 2 copper layers, 305.8 x 96.2 mm, 3 parts

Commit message: removed logo from keyboard plate design (janky Kicad fix + new Gerbers)
Parts:
- removed G***: LOGO, logos:coseyfannitutti_16mm
- removed G***: LOGO, logos:DISCIPLINE_SMALL_COPPER
- removed G***: LOGO, logos:DISCIPLINE_SMALL_MASK
Other:
- net class Default removed
- board text added: "1.2"
- board text added: "7/2/2019 - updated 1/2/2025"
- board text removed: "1.1"
- board text removed: "7/2/2019 - updated 12/3/2019"
